Commit message: fix(urdf): remove gripper offset when bracket is absent
Add has_bracket param to onrobot_rg2 macro. Without bracket,
joint0 xyz offset is zeroed so the gripper sits flush against
tool0. Camera bringup passes has_bracket:=true to preserve the
existing 4 mm offset.

Co-Authored-By: Claude Sonnet 4.6 <noreply@anthropic.com>

File: src/m0609_rg2_bringup/urdf/m0609_with_rg2_camera.urdf.xacro (robot description, xacro)
@@ -8,4 +8,4 @@
   <xacro:include filename="$(find m0609_rg2_bringup)/urdf/realsense_bracket.urdf.xacro"/>
   <!-- RG2 그리퍼를 tool0에 부착 -->
-  <xacro:onrobot_rg2 prefix="rg2_" effector_base="tool0"/>
+  <xacro:onrobot_rg2 prefix="rg2_" effector_base="tool0" has_bracket="true"/>
 </robot>

File: src/m0609_rg2_bringup/urdf/onrobot_rg2.xacro (robot description, xacro)
@@ -1,5 +1,5 @@
 <?xml version="1.0"?>
 <robot xmlns:xacro="http://ros.org/wiki/xacro">
-  <xacro:macro name="base_link" params="prefix effector_base:=world">
+  <xacro:macro name="base_link" params="prefix effector_base:=world has_bracket:=false">
     <link name="${prefix}base_link">
       <inertial>
@@ -31,5 +31,10 @@
         <parent link="${effector_base}"/>
         <child link="${prefix}base_link"/>
-        <origin xyz= "0.004 0. 0." rpy="1.5708 0 1.5708" />
+        <xacro:if value="${has_bracket}">
+          <origin xyz="0.004 0. 0." rpy="1.5708 0 1.5708" />
+        </xacro:if>
+        <xacro:unless value="${has_bracket}">
+          <origin xyz="0. 0. 0." rpy="1.5708 0 1.5708" />
+        </xacro:unless>
     </joint>
     <gazebo reference="${prefix}base_link">

File: src/m0609_rg2_bringup/urdf/onrobot_rg2_model_macro.xacro (robot description, xacro)
@@ -141,6 +141,6 @@
     <xacro:finger_joints prefix="${prefix}" fingerprefix="right" reflect="-1.0"/>
   </xacro:macro>
-  <xacro:macro name="onrobot_rg2" params="prefix effector_base:=world">
-    <xacro:base_link prefix="${prefix}" effector_base="${effector_base}"/>
+  <xacro:macro name="onrobot_rg2" params="prefix effector_base:=world has_bracket:=false">
+    <xacro:base_link prefix="${prefix}" effector_base="${effector_base}" has_bracket="${has_bracket}"/>
     <xacro:finger_links prefix="${prefix}" fingerprefix="left"/>
     <xacro:finger_links prefix="${prefix}" fingerprefix="right"/>
